File: docs/schematic/main_connection.kicad_sch (KiCad schematic)
At the start: 10 parts, among them J1 PJ-011A, J2 DIN-5, SW1 SW_SPST, SW2 SW_Push

Commit message: Dummy text removal; some tables and images
Connections:
- net +5V: no longer SW2.1
- net at DRV8833. (VCC): now also A1.D9
- net at DRV8833. (VCC): now also A1.D7
- net at DRV8833. (VCC): now also A1.D45; no longer TSS-110-05-F-D-RA1. (20)
- net at A1.A0: now also SW2.2
- net at A1.A8: now also SW2.1; no longer SW2.2
- new net: DRV8833. (VCC), DRV8833. (VCC), DRV8833. (VCC), J1.3
- new net: DRV8833. (VCC), DRV8833. (VCC), DRV8833. (VCC), SW1.2 (B)
- new net: DRV8833. (VCC), TSS-110-05-F-D-RA2. (20) (x6)
- new net: DRV8833. (VCC), TSS-110-05-F-D-RA1. (20) (x6)
Changed lines of the file:
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@@
 	(wire
 		(pts
-			(xy 158.75 133.35) (xy 181.61 133.35)
-		)
-		(stroke
-			(width 0)
-			(type default)
-		)
-	)
-	(wire
-		(pts
 			(xy 26.67 107.95) (xy 26.67 181.61)
 		)
@@
 	(wire
 		(pts
+			(xy 74.93 186.69) (xy 74.93 176.53)
+		)
+		(stroke
+			(width 0)
+			(type default)
+		)
+	)
+	(wire
+		(pts
 			(xy 16.51 66.04) (xy 38.1 66.04)
 		)
@@
 	(wire
 		(pts
+			(xy 161.29 133.35) (xy 181.61 133.35)
+		)
+		(stroke
+			(width 0)
+			(type default)
+		)
+	)
+	(wire
+		(pts
 			(xy 83.82 76.2) (xy 76.2 76.2)
 		)
@@
 	(wire
 		(pts
+			(xy 161.29 186.69) (xy 74.93 186.69)
+		)
+		(stroke
+			(width 0)
+			(type default)
+		)
+	)
+	(wire
+		(pts
 			(xy 200.66 62.23) (xy 200.66 77.47)
 		)
@@
 	(wire
 		(pts
-			(xy 181.61 116.84) (xy 181.61 119.38)
-		)
-		(stroke
-			(width 0)
-			(type default)
-		)
-	)
-	(wire
-		(pts
 			(xy 17.78 78.74) (xy 17.78 190.5)
 		)
@@
 	(wire
 		(pts
+			(xy 181.61 116.84) (xy 181.61 119.38)
+		)
+		(stroke
+			(width 0)
+			(type default)
+		)
+	)
+	(wire
+		(pts
 			(xy 87.63 194.31) (xy 171.45 194.31)
 		)
@@
 	(wire
 		(pts
+			(xy 161.29 133.35) (xy 161.29 186.69)
+		)
+		(stroke
+			(width 0)
+			(type default)
+		)
+	)
+	(wire
+		(pts
 			(xy 19.05 189.23) (xy 19.05 80.01)
 		)
@@
 	(wire
 		(pts
+			(xy 158.75 116.84) (xy 181.61 116.84)
+		)
+		(stroke
+			(width 0)
+			(type default)
+		)
+	)
+	(wire
+		(pts
 			(xy 54.61 110.49) (xy 54.61 97.79)
 		)
@@
 	(wire
 		(pts
-			(xy 158.75 133.35) (xy 158.75 186.69)
+			(xy 158.75 116.84) (xy 158.75 185.42)
 		)
 		(stroke
@@
 	(wire
 		(pts
-			(xy 95.25 186.69) (xy 95.25 176.53)
+			(xy 95.25 185.42) (xy 95.25 176.53)
 		)
 		(stroke
@@
 	(wire
 		(pts
-			(xy 158.75 186.69) (xy 95.25 186.69)
+			(xy 158.75 185.42) (xy 95.25 185.42)
 		)
 		(stroke
@@
 	)
 	(symbol
-		(lib_id "power:+5V")
-		(at 181.61 116.84 0)
-		(unit 1)
-		(exclude_from_sim no)
-		(in_bom yes)
-		(on_board yes)
-		(dnp no)
-		(fields_autoplaced yes)
-		(property "Reference" "#PWR013"
-			(at 181.61 120.65 0)
-			(effects
-				(font
-					(size 1.27 1.27)
-				)
-				(hide yes)
-			)
-		)
-		(property "Value" "+5V"
-			(at 181.61 111.76 0)
-			(effects
-				(font
-					(size 1.27 1.27)
-				)
-			)
-		)
-		(property "Footprint" ""
-			(at 181.61 116.84 0)
-			(effects
-				(font
-					(size 1.27 1.27)
-				)
-				(hide yes)
-			)
-		)
-		(property "Datasheet" ""
-			(at 181.61 116.84 0)
-			(effects
-				(font
-					(size 1.27 1.27)
-				)
-				(hide yes)
-			)
-		)
-		(property "Description" "Power symbol creates a global label with name \"+5V\""
-			(at 181.61 116.84 0)
-			(effects
-				(font
-					(size 1.27 1.27)
-				)
-				(hide yes)
-			)
-		)
-		(pin "1"
-		)
-		(instances
-			(project ""
-				(path "/31816756-201d-488d-8e24-e90bcff5bfd9"
-					(reference "#PWR013")
-					(unit 1)
-				)
-			)
-		)
-	)
-	(symbol
 		(lib_id "power:GND")
 		(at 187.96 146.05 90)
@@
 		(on_board yes)
 		(dnp no)
-		(fields_autoplaced yes)
 		(property "Reference" "SW2"
 			(at 185.42 123.1899 90)
